File: hardware/beepyRcBrd/3v3_external_reg.kicad_sch (KiCad schematic)
At the start: 4 parts, among them U9 TLV1117-33

Commit message: feat: completed beepyRcBrd_rev_0_0.pdf
Parts:
- added R21: 0, beepyRcBrd:R_0603_1608Metric_Pad0.98x0.95mm_HandSolder, symbol beepyRc_symbols:R
- C11, C5: footprint Capacitor_SMD:C_0603_1608Metric_Pad1.08x0.95mm_HandSolder -> beepyRcBrd:C_0603_1608Metric_Pad1.08x0.95mm_HandSolder
- D5: footprint Diode_SMD:D_SOD-323 -> beepyRcBrd:D_SOD-323
- U9: footprint lscs:SOT-223_L6.5-W3.5-P2.30-LS7.0-BR -> beepyRcBrd:SOT-223_L6.5-W3.5-P2.30-LS7.0-BR
Connections:
- net V_IN: now also R21.1; no longer C5.1, D5.1 (K), U9.3 (VI)
- net V_OUT: now also U9.4 (VO)
- new net: C5.1, D5.1 (K), R21.2, U9.3 (VI)
Changed lines of the file:
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@@
 		(rev "V0.0")
 		(company "ElectronPlant")
+		(comment 1 "© David Arnaiz 2026")
+		(comment 2 "Licensed under CERN-OHL-S v2")
 	)
 	(text "3.3V @500mA\n(thermally limited)"
@@
 	(text "BeepyRC"
 		(exclude_from_sim no)
-		(at 233.68 173.736 0)
+		(at 252.222 173.99 0)
 		(effects
 			(font
@@
 	)
 	(junction
+		(at 162.56 80.01)
+		(diameter 0)
+		(color 0 0 0 0)
+	)
+	(junction
 		(at 176.53 80.01)
 		(diameter 0)
@@
 	(wire
 		(pts
+			(xy 162.56 80.01) (xy 176.53 80.01)
+		)
+		(stroke
+			(width 0)
+			(type default)
+		)
+	)
+	(wire
+		(pts
 			(xy 125.73 95.25) (xy 151.13 95.25)
 		)
@@
 	(wire
 		(pts
+			(xy 162.56 82.55) (xy 162.56 80.01)
+		)
+		(stroke
+			(width 0)
+			(type default)
+		)
+	)
+	(wire
+		(pts
+			(xy 107.95 80.01) (xy 125.73 80.01)
+		)
+		(stroke
+			(width 0)
+			(type default)
+		)
+	)
+	(wire
+		(pts
 			(xy 176.53 92.71) (xy 176.53 95.25)
 		)
@@
 	(wire
 		(pts
-			(xy 158.75 80.01) (xy 176.53 80.01)
-		)
-		(stroke
-			(width 0)
-			(type default)
-		)
-	)
-	(wire
-		(pts
-			(xy 88.9 80.01) (xy 125.73 80.01)
+			(xy 158.75 80.01) (xy 162.56 80.01)
 		)
 		(stroke
@@
 	(wire
 		(pts
+			(xy 158.75 82.55) (xy 162.56 82.55)
+		)
+		(stroke
+			(width 0)
+			(type default)
+		)
+	)
+	(wire
+		(pts
 			(xy 151.13 87.63) (xy 151.13 95.25)
 		)
@@
 		(pts
 			(xy 176.53 80.01) (xy 214.63 80.01)
+		)
+		(stroke
+			(width 0)
+			(type default)
+		)
+	)
+	(wire
+		(pts
+			(xy 88.9 80.01) (xy 100.33 80.01)
 		)
 		(stroke
@@
 			)
 		)
-		(property "Footprint" "Capacitor_SMD:C_0603_1608Metric_Pad1.08x0.95mm_HandSolder"
+		(property "Footprint" "beepyRcBrd:C_0603_1608Metric_Pad1.08x0.95mm_HandSolder"
 			(at 126.6952 92.71 0)
 			(effects
@@
 				(path "/c17d25e0-24c9-466a-aee2-e4b5dcf71363/25416242-1327-4080-bdb9-7e497d324eea/def325ff-e16e-4cf4-9ff1-0efa69108464"
 					(reference "C5")
+					(unit 1)
+				)
+			)
+		)
+	)
+	(symbol
+		(lib_id "beepyRc_symbols:R")
+		(at 104.14 80.01 90)
+		(unit 1)
+		(exclude_from_sim no)
+		(in_bom yes)
+		(on_board yes)
+		(dnp no)
+		(property "Reference" "R21"
+			(at 99.314 78.74 90)
+			(effects
+				(font
+					(size 1.27 1.27)
+				)
+			)
+		)
+		(property "Value" "0"
+			(at 107.696 78.74 90)
+			(effects
+				(font
+					(size 1.27 1.27)
+				)
+			)
+		)
+		(property "Footprint" "beepyRcBrd:R_0603_1608Metric_Pad0.98x0.95mm_HandSolder"
+			(at 104.14 81.788 90)
+			(effects
+				(font
+					(size 1.27 1.27)
+				)
+				(hide yes)
+			)
+		)
+		(property "Datasheet" "~"
+			(at 104.14 80.01 0)
+			(effects
+				(font
+					(size 1.27 1.27)
+				)
+				(hide yes)
+			)
+		)
+		(property "Description" "Resistor"
+			(at 104.14 80.01 0)
+			(effects
+				(font
+					(size 1.27 1.27)
+				)
+				(hide yes)
+			)
+		)
+		(property "Sim.Device" ""
+			(at 104.14 80.01 0)
+			(effects
+				(font
+					(size 1.27 1.27)
+				)
+				(hide yes)
+			)
+		)
+		(property "Sim.Type" ""
+			(at 104.14 80.01 0)
+			(effects
+				(font
+					(size 1.27 1.27)
+				)
+				(hide yes)
+			)
+		)
+		(pin "2"
+		)
+		(pin "1"
+		)
+		(instances
+			(project "beepyRcBrd"
+				(path "/c17d25e0-24c9-466a-aee2-e4b5dcf71363/25416242-1327-4080-bdb9-7e497d324eea/def325ff-e16e-4cf4-9ff1-0efa69108464"
+					(reference "R21")
 					(unit 1)
 				)
@@
 			)
 		)
-		(property "Footprint" "Capacitor_SMD:C_0603_1608Metric_Pad1.08x0.95mm_HandSolder"
+		(property "Footprint" "beepyRcBrd:C_0603_1608Metric_Pad1.08x0.95mm_HandSolder"
 			(at 177.4952 92.71 0)
 			(effects
@@
 			)
 		)
-		(property "Footprint" "lscs:SOT-223_L6.5-W3.5-P2.30-LS7.0-BR"
+		(property "Footprint" "beepyRcBrd:SOT-223_L6.5-W3.5-P2.30-LS7.0-BR"
 			(at 151.13 80.01 0)
 			(effects
@@
 		)
 		(pin "2"
+		)
+		(pin "4"
 		)
 		(instances
@@
 			)
 		)
-		(property "Footprint" "Diode_SMD:D_SOD-323"
+		(property "Footprint" "beepyRcBrd:D_SOD-323"
 			(at 151.13 64.77 0)
 			(effects
