File: hardware/beepyRcBrd/3v_reg.kicad_sch (KiCad schematic)
At the start: 3 parts, among them U5 MC33275ST-3.3T3G

Commit message: feat: completed beepyRcBrd_rev_0_0.pdf
Parts:
- C3, C4: footprint Capacitor_SMD:C_0603_1608Metric_Pad1.08x0.95mm_HandSolder -> beepyRcBrd:C_0603_1608Metric_Pad1.08x0.95mm_HandSolder
- U5: footprint lscs:SOT-223_L6.5-W3.5-P2.30-LS7.0-BR -> beepyRcBrd:SOT-223_L6.5-W3.5-P2.30-LS7.0-BR
Changed lines of the file:
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@@
 		(rev "V0.0")
 		(company "ElectronPlant")
+		(comment 1 "© David Arnaiz 2026")
+		(comment 2 "Licensed under CERN-OHL-S v2")
 	)
 	(text "BeepyRC"
 		(exclude_from_sim no)
-		(at 230.632 173.99 0)
+		(at 252.476 173.736 0)
 		(effects
 			(font
@@
 			)
 		)
-		(property "Footprint" "Capacitor_SMD:C_0603_1608Metric_Pad1.08x0.95mm_HandSolder"
+		(property "Footprint" "beepyRcBrd:C_0603_1608Metric_Pad1.08x0.95mm_HandSolder"
 			(at 115.2652 99.06 0)
 			(effects
@@
 			)
 		)
-		(property "Footprint" "lscs:SOT-223_L6.5-W3.5-P2.30-LS7.0-BR"
+		(property "Footprint" "beepyRcBrd:SOT-223_L6.5-W3.5-P2.30-LS7.0-BR"
 			(at 140.97 95.25 0)
 			(effects
@@
 			)
 		)
-		(property "Footprint" "Capacitor_SMD:C_0603_1608Metric_Pad1.08x0.95mm_HandSolder"
+		(property "Footprint" "beepyRcBrd:C_0603_1608Metric_Pad1.08x0.95mm_HandSolder"
 			(at 166.0652 99.06 0)
 			(effects
