File: hardware/beepyRcBrd/bat_mon.kicad_sch (KiCad schematic)
At the start: 7 parts, among them U3 INA139

Commit message: fix: passing schematics ERC rules
Changed lines of the file:
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@@
+	)
+	(junction
+		(at 67.31 73.66)
+		(diameter 0)
+		(color 0 0 0 0)
 	)
 	(junction
@@
 	(wire
 		(pts
-			(xy 63.5 73.66) (xy 82.55 73.66)
+			(xy 63.5 73.66) (xy 67.31 73.66)
+		)
+		(stroke
+			(width 0)
+			(type default)
+		)
+	)
+	(wire
+		(pts
+			(xy 67.31 73.66) (xy 82.55 73.66)
 		)
 		(stroke
@@
 					(unit 1)
 				)
+			)
+		)
+	)
+	(symbol
+		(lib_id "beepyRc_symbols:PWR_FLAG")
+		(at 67.31 73.66 0)
+		(unit 1)
+		(exclude_from_sim no)
+		(in_bom yes)
+		(on_board yes)
+		(dnp no)
+		(property "Reference" "#FLG06"
+			(at 67.31 71.755 0)
+			(effects
+				(font
+					(size 1.27 1.27)
+				)
+				(hide yes)
+			)
+		)
+		(property "Value" "PWR_FLAG"
+			(at 67.31 69.596 0)
+			(effects
+				(font
+					(size 1.27 1.27)
+				)
+			)
+		)
+		(property "Footprint" ""
+			(at 67.31 73.66 0)
+			(effects
+				(font
+					(size 1.27 1.27)
+				)
+				(hide yes)
+			)
+		)
+		(property "Datasheet" "~"
+			(at 67.31 73.66 0)
+			(effects
+				(font
+					(size 1.27 1.27)
+				)
+				(hide yes)
+			)
+		)
+		(property "Description" "Special symbol for telling ERC where power comes from"
+			(at 67.31 73.66 0)
+			(effects
+				(font
+					(size 1.27 1.27)
+				)
+				(hide yes)
+			)
+		)
+		(pin "1"
+		)
+		(instances
+			(project ""
+				(path "/c17d25e0-24c9-466a-aee2-e4b5dcf71363/25416242-1327-4080-bdb9-7e497d324eea/f7650829-a817-41d0-84d7-b7cf65a2545c"
+					(reference "#FLG06")
+					(unit 1)
+				)

Commit message: feat: completed beepyRcBrd_rev_0_0.pdf
Parts:
- C1, C2: footprint Capacitor_SMD:C_0603_1608Metric_Pad1.08x0.95mm_HandSolder -> beepyRcBrd:C_0603_1608Metric_Pad1.08x0.95mm_HandSolder
- R11: footprint Resistor_SMD:R_0603_1608Metric_Pad0.98x0.95mm_HandSolder -> beepyRcBrd:R_0603_1608Metric_Pad0.98x0.95mm_HandSolder
- R42: renamed from R_SENSE1; footprint Resistor_SMD:R_0603_1608Metric_Pad0.98x0.95mm_HandSolder -> beepyRcBrd:R_0603_1608Metric_Pad0.98x0.95mm_HandSolder
- R43: renamed from R_SENSE2; footprint Resistor_SMD:R_0603_1608Metric_Pad0.98x0.95mm_HandSolder -> beepyRcBrd:R_0603_1608Metric_Pad0.98x0.95mm_HandSolder
- Rs1: footprint Resistor_SMD:R_1206_3216Metric_Pad1.30x1.75mm_HandSolder -> beepyRcBrd:R_1206_3216Metric_Pad1.30x1.75mm_HandSolder
- U3: footprint Package_TO_SOT_SMD:SOT-23-5 -> beepyRcBrd:SOT-23-5
Changed lines of the file:
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@@
 		(rev "V0.0")
 		(company "Electron Plant")
+		(comment 1 "© David Arnaiz 2026")
+		(comment 2 "Licensed under CERN-OHL-S v2")
 	)
 	(text "V_BAT_MEAS = 0.24 * V_BAT"
@@
 	(text "BeepyRC"
 		(exclude_from_sim no)
-		(at 235.712 173.99 0)
+		(at 252.476 174.498 0)
 		(effects
 			(font
@@
 		(dnp no)
 		(fields_autoplaced yes)
-		(property "Reference" "R_SENSE1"
+		(property "Reference" "R42"
 			(at 85.09 83.8199 0)
 			(effects
@@
 			)
 		)
-		(property "Footprint" "Resistor_SMD:R_0603_1608Metric_Pad0.98x0.95mm_HandSolder"
+		(property "Footprint" "beepyRcBrd:R_0603_1608Metric_Pad0.98x0.95mm_HandSolder"
 			(at 80.772 85.09 90)
 			(effects
@@
 			(project "beepyRcBrd"
 				(path "/c17d25e0-24c9-466a-aee2-e4b5dcf71363/25416242-1327-4080-bdb9-7e497d324eea/f7650829-a817-41d0-84d7-b7cf65a2545c"
-					(reference "R_SENSE1")
+					(reference "R42")
 					(unit 1)
 				)
@@
 			)
 		)
-		(property "Footprint" "Capacitor_SMD:C_0603_1608Metric_Pad1.08x0.95mm_HandSolder"
+		(property "Footprint" "beepyRcBrd:C_0603_1608Metric_Pad1.08x0.95mm_HandSolder"
 			(at 102.5652 105.41 0)
 			(effects
@@
 			)
 		)
-		(property "Footprint" "Package_TO_SOT_SMD:SOT-23-5"
+		(property "Footprint" "beepyRcBrd:SOT-23-5"
 			(at 154.94 45.72 0)
 			(effects
@@
 		(dnp no)
 		(fields_autoplaced yes)
-		(property "Reference" "R_SENSE2"
+		(property "Reference" "R43"
 			(at 85.09 100.3299 0)
 			(effects
@@
 			)
 		)
-		(property "Footprint" "Resistor_SMD:R_0603_1608Metric_Pad0.98x0.95mm_HandSolder"
+		(property "Footprint" "beepyRcBrd:R_0603_1608Metric_Pad0.98x0.95mm_HandSolder"
 			(at 80.772 101.6 90)
 			(effects
@@
 			(project "beepyRcBrd"
 				(path "/c17d25e0-24c9-466a-aee2-e4b5dcf71363/25416242-1327-4080-bdb9-7e497d324eea/f7650829-a817-41d0-84d7-b7cf65a2545c"
-					(reference "R_SENSE2")
+					(reference "R43")
 					(unit 1)
 				)
@@
 			)
 		)
-		(property "Footprint" "Capacitor_SMD:C_0603_1608Metric_Pad1.08x0.95mm_HandSolder"
+		(property "Footprint" "beepyRcBrd:C_0603_1608Metric_Pad1.08x0.95mm_HandSolder"
 			(at 191.4652 55.88 0)
 			(effects
@@
 			)
 		)
-		(property "Footprint" "Resistor_SMD:R_1206_3216Metric_Pad1.30x1.75mm_HandSolder"
+		(property "Footprint" "beepyRcBrd:R_1206_3216Metric_Pad1.30x1.75mm_HandSolder"
 			(at 125.73 75.438 90)
 			(effects
@@
 			)
 		)
-		(property "Footprint" "Resistor_SMD:R_0603_1608Metric_Pad0.98x0.95mm_HandSolder"
+		(property "Footprint" "beepyRcBrd:R_0603_1608Metric_Pad0.98x0.95mm_HandSolder"
 			(at 176.022 52.07 90)
 			(effects
