File: hardware/beepyRcBrd/beepyRcBrd.kicad_pcb (KiCad board)
At the start: 4 copper layers, 0 parts

Commit message: feat: completed beepyRcBrd_rev_0_0.pdf
Parts:
- added BUZZER1: TMB12A05, beepyRcBrd:BUZ-TH_BD12.0-P7.60-D0.6-FD, F.Cu at (118.2, 70.5)
- added C1: 5.1nF, beepyRcBrd:C_0603_1608Metric_Pad1.08x0.95mm_HandSolder, B.Cu at (78.2, 124.0)
- added C10: 22μF, beepyRcBrd:C_0603_1608Metric_Pad1.08x0.95mm_HandSolder, F.Cu at (87.5, 126.0)
- added C11: 1μF, beepyRcBrd:C_0603_1608Metric_Pad1.08x0.95mm_HandSolder, B.Cu at (88.2, 137.9)
- added C12: 10nF, beepyRcBrd:C_0603_1608Metric_Pad1.08x0.95mm_HandSolder, B.Cu at (76.2, 107.0)
- added C13: 10nF, beepyRcBrd:C_0603_1608Metric_Pad1.08x0.95mm_HandSolder, B.Cu at (76.2, 109.0)
- added C14: 22μF, beepyRcBrd:C_0603_1608Metric_Pad1.08x0.95mm_HandSolder, B.Cu at (85.7, 88.0)
- added C15: 30pF, beepyRcBrd:C_0603_1608Metric_Pad1.08x0.95mm_HandSolder, F.Cu at (104.5, 97.7)
- added C16: 14pF, beepyRcBrd:C_0603_1608Metric_Pad1.08x0.95mm_HandSolder, F.Cu at (103.5, 84.8)
- added C17: 30pF, beepyRcBrd:C_0603_1608Metric_Pad1.08x0.95mm_HandSolder, F.Cu at (104.5, 103.0)
- added C18: 14pF, beepyRcBrd:C_0603_1608Metric_Pad1.08x0.95mm_HandSolder, F.Cu at (103.5, 88.8)
- added C19: 4.7μF, beepyRcBrd:C_0603_1608Metric_Pad1.08x0.95mm_HandSolder, F.Cu at (121.2, 103.0)
- added C2: 18nF, beepyRcBrd:C_0603_1608Metric_Pad1.08x0.95mm_HandSolder, B.Cu at (83.5, 119.4)
- added C20: 10μF, beepyRcBrd:C_0603_1608Metric_Pad1.08x0.95mm_HandSolder, B.Cu at (111.0, 103.0)
- added C21: 100nF, beepyRcBrd:C_0603_1608Metric_Pad1.08x0.95mm_HandSolder, B.Cu at (120.4, 96.7)
- added C22: 100nF, beepyRcBrd:C_0603_1608Metric_Pad1.08x0.95mm_HandSolder, B.Cu at (115.1, 96.8)
- added C23: 100nF, beepyRcBrd:C_0603_1608Metric_Pad1.08x0.95mm_HandSolder, F.Cu at (104.2, 144.5)
- added C24: 100nF, beepyRcBrd:C_0603_1608Metric_Pad1.08x0.95mm_HandSolder, B.Cu at (120.4, 90.9)
- added C25: 100nF, beepyRcBrd:C_0603_1608Metric_Pad1.08x0.95mm_HandSolder, B.Cu at (111.3, 88.3)
- added C26: 100nF, beepyRcBrd:C_0603_1608Metric_Pad1.08x0.95mm_HandSolder, B.Cu at (114.7, 90.4)
- added C27: 1μF, beepyRcBrd:C_0603_1608Metric_Pad1.08x0.95mm_HandSolder, B.Cu at (111.0, 97.0)
- added C28: 100nF, beepyRcBrd:C_0603_1608Metric_Pad1.08x0.95mm_HandSolder, B.Cu at (111.0, 99.0)
- added C29: 22μF, beepyRcBrd:C_0603_1608Metric_Pad1.08x0.95mm_HandSolder, B.Cu at (85.7, 86.0)
- added C3: 1μF, beepyRcBrd:C_0603_1608Metric_Pad1.08x0.95mm_HandSolder, B.Cu at (74.5, 142.0)
- added C30: 100nF, beepyRcBrd:C_0603_1608Metric_Pad1.08x0.95mm_HandSolder, B.Cu at (78.2, 80.0)
- added C33: 100nF, beepyRcBrd:C_0603_1608Metric_Pad1.08x0.95mm_HandSolder, F.Cu at (81.2, 77.5)
- added C34: 100nF, beepyRcBrd:C_0603_1608Metric_Pad1.08x0.95mm_HandSolder, F.Cu at (88.7, 85.0)
- added C37: 100nF, beepyRcBrd:C_0603_1608Metric_Pad1.08x0.95mm_HandSolder, F.Cu at (81.2, 81.5)
- added C4: 1μF, beepyRcBrd:C_0603_1608Metric_Pad1.08x0.95mm_HandSolder, B.Cu at (70.5, 142.0)
- added C5: 1μF, beepyRcBrd:C_0603_1608Metric_Pad1.08x0.95mm_HandSolder, B.Cu at (84.0, 141.5)
- added C6: 10μF, beepyRcBrd:C_0603_1608Metric_Pad1.08x0.95mm_HandSolder, F.Cu at (79.0, 110.0)
- added C7: 10μF, beepyRcBrd:C_0603_1608Metric_Pad1.08x0.95mm_HandSolder, F.Cu at (75.0, 110.0)
- added C8: 100nF, beepyRcBrd:C_0603_1608Metric_Pad1.08x0.95mm_HandSolder, F.Cu at (77.0, 110.0)
- added C9: 22μF, beepyRcBrd:C_0603_1608Metric_Pad1.08x0.95mm_HandSolder, F.Cu at (87.5, 124.0)
- added D1: RED, beepyRcBrd:LED_0603_1608Metric_Pad1.05x0.95mm_HandSolder, F.Cu at (83.2, 154.1)
- added D10: UESD3.3DT5G, beepyRcBrd:SOT-723_L1.2-W0.8-P0.40-LS1.2-BR, F.Cu at (94.6, 48.9)
- added D11: UESD3.3DT5G, beepyRcBrd:SOT-723_L1.2-W0.8-P0.40-LS1.2-BR, F.Cu at (98.1, 48.9)
- added D12: UESD3.3DT5G, beepyRcBrd:SOT-723_L1.2-W0.8-P0.40-LS1.2-BR, B.Cu at (94.7, 65.0)
- added D13: UESD3.3DT5G, beepyRcBrd:SOT-723_L1.2-W0.8-P0.40-LS1.2-BR, B.Cu at (98.0, 65.0)
- added D14: UESD3.3DT5G, beepyRcBrd:SOT-723_L1.2-W0.8-P0.40-LS1.2-BR, B.Cu at (103.4, 118.0)
- added D15: UESD3.3DT5G, beepyRcBrd:SOT-723_L1.2-W0.8-P0.40-LS1.2-BR, B.Cu at (107.0, 118.0)
- added D2: GREEN, beepyRcBrd:LED_0603_1608Metric_Pad1.05x0.95mm_HandSolder, F.Cu at (70.7, 154.1)
- added D3: YELLOW, beepyRcBrd:LED_0603_1608Metric_Pad1.05x0.95mm_HandSolder, F.Cu at (76.7, 154.1)
- added D4: SDM20E40C-7-F, beepyRcBrd:SOT-23-3_L2.9-W1.6-P1.90-LS2.8-BR, F.Cu at (92.8, 112.8)
- added D5: D_Schottky, beepyRcBrd:D_SOD-323, B.Cu at (90.2, 138.2)
- added D6: CDSOT23-SM712, beepyRcBrd:SOT-23_L2.9-W1.3-P1.90-LS2.4-BR, B.Cu at (134.4, 102.0)
- added D7: SMBJ15A_C83846, beepyRcBrd:SMB_L4.6-W3.6-LS5.3-RD, F.Cu at (68.7, 112.1)
- added D8: CDSOT23-SM712, beepyRcBrd:SOT-23_L2.9-W1.3-P1.90-LS2.4-BR, B.Cu at (129.7, 102.0)
- added D9: UESD3.3DT5G, beepyRcBrd:SOT-723_L1.2-W0.8-P0.40-LS1.2-BR, B.Cu at (61.1, 106.1)
- added F1: MINISMDC050F-2, beepyRcBrd:Fuse_1812_4532Metric_Pad1.30x3.40mm_HandSolder, B.Cu at (133.7, 87.5)
- added F2: BSMD1812L-600-12V, beepyRcBrd:Fuse_1812_4532Metric_Pad1.30x3.40mm_HandSolder, F.Cu at (68.5, 118.5)
- added FB1: FerriteBead, beepyRcBrd:R_0603_1608Metric_Pad0.98x0.95mm_HandSolder, F.Cu at (87.5, 120.0)
- added FB2: FerriteBead, beepyRcBrd:R_0603_1608Metric_Pad0.98x0.95mm_HandSolder, B.Cu at (111.0, 101.0)
- added G***: LOGO, beepyRcBrd:LOGO, B.Cu at (117.3, 38.8)
- added H1: MT, beepyRcBrd:MountingHole_4.3mm_M4_DIN965_Pad_TopBottom, F.Cu at (57.2, 36.0)
- added H10: MT, beepyRcBrd:MountingHole_2.2mm_M2_DIN965_Pad_TopBottom, F.Cu at (65.4, 147.1)
- added H11: MT, beepyRcBrd:MountingHole_2.2mm_M2_DIN965_Pad_TopBottom, F.Cu at (128.0, 127.9)
- added H12: MT, beepyRcBrd:MountingHole_2.2mm_M2_DIN965_Pad_TopBottom, F.Cu at (128.0, 147.1)
- added H13: MT, beepyRcBrd:MountingHole_4.3mm_M4_DIN965_Pad_TopBottom, F.Cu at (63.3, 84.1)
- added H14: MT, beepyRcBrd:MountingHole_4.3mm_M4_DIN965_Pad_TopBottom, F.Cu at (63.3, 70.0)
- added H2: MT, beepyRcBrd:MountingHole_4.3mm_M4_DIN965_Pad_TopBottom, F.Cu at (136.2, 36.0)
- added H3: MT, beepyRcBrd:MountingHole_4.3mm_M4_DIN965_Pad_TopBottom, F.Cu at (57.2, 154.0)
- added H4: MT, beepyRcBrd:MountingHole_4.3mm_M4_DIN965_Pad_TopBottom, F.Cu at (136.2, 154.0)
- added H5: MT, beepyRcBrd:MountingHole_2.2mm_M2_DIN965_Pad_TopBottom, F.Cu at (65.3, 42.9)
- added H6: MT, beepyRcBrd:MountingHole_2.2mm_M2_DIN965_Pad_TopBottom, F.Cu at (65.4, 62.1)
- added H7: MT, beepyRcBrd:MountingHole_2.2mm_M2_DIN965_Pad_TopBottom, F.Cu at (128.0, 42.9)
- added H8: MT, beepyRcBrd:MountingHole_2.2mm_M2_DIN965_Pad_TopBottom, F.Cu at (128.1, 62.1)
- added H9: MT, beepyRcBrd:MountingHole_2.2mm_M2_DIN965_Pad_TopBottom, F.Cu at (65.3, 127.9)
- added J1: Conn_01x06, beepyRcBrd:PinHeader_1x06_P2.54mm_Vertical, F.Cu at (91.1, 57.8)
- added J10: Conn_01x03, beepyRcBrd:PinHeader_1x03_P2.54mm_Vertical, F.Cu at (91.6, 36.9)
- added J11: Conn_01x03, beepyRcBrd:PinHeader_1x03_P2.54mm_Vertical, F.Cu at (96.1, 36.8)
- added J14: Conn_01x04, beepyRcBrd:PinHeader_1x04_P2.54mm_Vertical, F.Cu at (76.1, 32.0)
- added J15: Conn_01x04, beepyRcBrd:PinHeader_1x04_P2.54mm_Vertical, F.Cu at (83.8, 94.4)
- added J16: Conn_01x03, beepyRcBrd:rc, F.Cu at (90.3, 131.6)
- added J17: Conn_01x02, beepyRcBrd:PinHeader_1x02_P2.54mm_Vertical, F.Cu at (78.8, 97.0)
- added J18: Conn_01x04, beepyRcBrd:PinHeader_1x04_P2.54mm_Vertical, F.Cu at (53.7, 96.0)
- added J19: Conn_01x05, beepyRcBrd:CONN-TH_5P-P3.50_DORABO_DB125-3.5-5P-GN-S, F.Cu at (137.5, 114.0)
- added J2: Conn_01x06, beepyRcBrd:PinHeader_1x06_P2.54mm_Vertical, F.Cu at (102.2, 57.8)
- added J20: Conn_01x04, beepyRcBrd:PinHeader_1x04_P2.54mm_Vertical, F.Cu at (90.5, 147.5)
- added J3: Conn_01x06, beepyRcBrd:PinHeader_1x06_P2.54mm_Vertical, F.Cu at (140.5, 68.7)
- added J4: Conn_01x06, beepyRcBrd:PinHeader_1x06_P2.54mm_Vertical, F.Cu at (140.2, 87.8)
- added J5: Conn_01x06, beepyRcBrd:PinHeader_1x06_P2.54mm_Vertical, F.Cu at (98.9, 113.1)
- added J6: Conn_01x06, beepyRcBrd:PinHeader_1x06_P2.54mm_Vertical, F.Cu at (111.4, 113.1)
- added J7: Conn_01x02, beepyRcBrd:CONN-TH_P5.00_KF301-5.0-2P, F.Cu at (60.7, 116.1)
- added J8: Conn_01x08, beepyRcBrd:gy91, F.Cu at (53.7, 86.2)
- added J9: Conn_01x03, beepyRcBrd:PinHeader_1x03_P2.54mm_Vertical, F.Cu at (100.6, 36.8)
- added L2: 1.8μH, beepyRcBrd:IND-SMD_L7.0-W6.6_MCW-0650-220, F.Cu at (81.8, 119.5)
- added Motor1: Motor, beepyRcBrd:Motor, F.Cu at (65.2, 52.5)
- added Motor2: Motor, beepyRcBrd:Motor, F.Cu at (128.2, 52.5)
- added Motor3: Motor, beepyRcBrd:Motor, F.Cu at (65.2, 137.5)
- added Motor4: Motor, beepyRcBrd:Motor, F.Cu at (128.2, 137.4)
- added Q1: BSS138LT1G, beepyRcBrd:SOT-23-3_L2.9-W1.6-P1.90-LS2.8-BR, B.Cu at (75.5, 41.4)
- added Q2: BSS138LT1G, beepyRcBrd:SOT-23-3_L2.9-W1.6-P1.90-LS2.8-BR, B.Cu at (112.4, 76.0)
- added Q3: BSS138DW-7-F, beepyRcBrd:SC-70-6_L2.2-W1.3-P0.65-LS2.1-TL, B.Cu at (98.4, 107.7)
- added Q4: BSS138LT1G, beepyRcBrd:SOT-23-3_L2.9-W1.6-P1.90-LS2.8-BR, B.Cu at (96.3, 138.5)
- added Q5: BSS138LT1G, beepyRcBrd:SOT-23-3_L2.9-W1.6-P1.90-LS2.8-BR, B.Cu at (75.5, 47.0)
- added R1: 10k, beepyRcBrd:R_0603_1608Metric_Pad0.98x0.95mm_HandSolder, B.Cu at (62.7, 78.0)
- added R10: 51k, beepyRcBrd:R_0603_1608Metric_Pad0.98x0.95mm_HandSolder, B.Cu at (82.7, 111.0)
- added R11: 30k, beepyRcBrd:R_0603_1608Metric_Pad0.98x0.95mm_HandSolder, B.Cu at (78.2, 122.0)
- added R12: 51k, beepyRcBrd:R_0603_1608Metric_Pad0.98x0.95mm_HandSolder, B.Cu at (76.2, 110.9)
- added R13: 0, beepyRcBrd:R_0603_1608Metric_Pad0.98x0.95mm_HandSolder, B.Cu at (130.2, 79.5)
- added R14: 10k, beepyRcBrd:R_0603_1608Metric_Pad0.98x0.95mm_HandSolder, F.Cu at (117.4, 84.0)
- added R15: 0, beepyRcBrd:R_0603_1608Metric_Pad0.98x0.95mm_HandSolder, B.Cu at (130.1, 75.0)
- added R16: 10k, beepyRcBrd:R_0603_1608Metric_Pad0.98x0.95mm_HandSolder, B.Cu at (115.7, 132.0)
- added R17: 51R, beepyRcBrd:R_0603_1608Metric_Pad0.98x0.95mm_HandSolder, B.Cu at (81.5, 40.0)
- added R18: 51R, beepyRcBrd:R_0603_1608Metric_Pad0.98x0.95mm_HandSolder, B.Cu at (84.0, 40.0)
- added R19: 10k, beepyRcBrd:R_0603_1608Metric_Pad0.98x0.95mm_HandSolder, B.Cu at (99.3, 81.3)
- added R2: 2.2k, beepyRcBrd:R_0603_1608Metric_Pad0.98x0.95mm_HandSolder, F.Cu at (81.2, 154.1)
- added R20: 10k, beepyRcBrd:R_0603_1608Metric_Pad0.98x0.95mm_HandSolder, B.Cu at (96.5, 142.5)
- added R21: 0, beepyRcBrd:R_0603_1608Metric_Pad0.98x0.95mm_HandSolder, B.Cu at (80.5, 145.5)
- added R23: 22R, beepyRcBrd:R_0603_1608Metric_Pad0.98x0.95mm_HandSolder, B.Cu at (89.8, 81.0)
- added R24: 22R, beepyRcBrd:R_0603_1608Metric_Pad0.98x0.95mm_HandSolder, B.Cu at (105.7, 94.0)
- added R25: 22R, beepyRcBrd:R_0603_1608Metric_Pad0.98x0.95mm_HandSolder, B.Cu at (128.0, 94.0)
- added R26: 22R, beepyRcBrd:R_0603_1608Metric_Pad0.98x0.95mm_HandSolder, B.Cu at (62.7, 76.0)
- added R27: 0, beepyRcBrd:R_0603_1608Metric_Pad0.98x0.95mm_HandSolder, B.Cu at (61.2, 97.0)
- added R28: 0, beepyRcBrd:R_0603_1608Metric_Pad0.98x0.95mm_HandSolder, B.Cu at (61.2, 101.5)
- added R29: 10k, beepyRcBrd:R_0603_1608Metric_Pad0.98x0.95mm_HandSolder, B.Cu at (63.5, 107.5)
- added R3: 2.2k, beepyRcBrd:R_0603_1608Metric_Pad0.98x0.95mm_HandSolder, F.Cu at (74.8, 154.1)
- added R30: 10k, beepyRcBrd:R_0603_1608Metric_Pad0.98x0.95mm_HandSolder, B.Cu at (58.5, 107.5)
- added R31: 100R, beepyRcBrd:R_0603_1608Metric_Pad0.98x0.95mm_HandSolder, B.Cu at (120.2, 78.5)
- added R32: 200k, beepyRcBrd:R_0603_1608Metric_Pad0.98x0.95mm_HandSolder, F.Cu at (107.5, 88.9)
- added R33: 75R, beepyRcBrd:R_0603_1608Metric_Pad0.98x0.95mm_HandSolder, B.Cu at (78.2, 82.0)
- added R34: 75R, beepyRcBrd:R_0603_1608Metric_Pad0.98x0.95mm_HandSolder, B.Cu at (85.7, 90.2)
- added R35: 10k, beepyRcBrd:R_0603_1608Metric_Pad0.98x0.95mm_HandSolder, B.Cu at (115.7, 134.0)
- added R36: 10k, beepyRcBrd:R_0603_1608Metric_Pad0.98x0.95mm_HandSolder, B.Cu at (108.2, 132.0)
- added R37: 10k, beepyRcBrd:R_0603_1608Metric_Pad0.98x0.95mm_HandSolder, B.Cu at (108.2, 134.0)
- added R38: 10k, beepyRcBrd:R_0603_1608Metric_Pad0.98x0.95mm_HandSolder, B.Cu at (113.2, 65.0)
- added R39: 10k, beepyRcBrd:R_0603_1608Metric_Pad0.98x0.95mm_HandSolder, B.Cu at (113.2, 62.5)
- added R4: 2.2k, beepyRcBrd:R_0603_1608Metric_Pad0.98x0.95mm_HandSolder, F.Cu at (68.7, 154.1)
- added R40: 10k, beepyRcBrd:R_0603_1608Metric_Pad0.98x0.95mm_HandSolder, B.Cu at (78.5, 65.0)
- added R41: 10k, beepyRcBrd:R_0603_1608Metric_Pad0.98x0.95mm_HandSolder, B.Cu at (78.5, 63.0)
- added R42: 40k, beepyRcBrd:R_0603_1608Metric_Pad0.98x0.95mm_HandSolder, B.Cu at (83.5, 115.4)
- added R43: 10k, beepyRcBrd:R_0603_1608Metric_Pad0.98x0.95mm_HandSolder, B.Cu at (83.5, 117.4)
- added R44: 50k, beepyRcBrd:R_0603_1608Metric_Pad0.98x0.95mm_HandSolder, B.Cu at (82.7, 107.0)
- added R45: 10k, beepyRcBrd:R_0603_1608Metric_Pad0.98x0.95mm_HandSolder, B.Cu at (76.2, 105.0)
- added R5: 10k, beepyRcBrd:R_0603_1608Metric_Pad0.98x0.95mm_HandSolder, F.Cu at (105.1, 138.5)
- added R6: 10k, beepyRcBrd:R_0603_1608Metric_Pad0.98x0.95mm_HandSolder, F.Cu at (106.1, 136.0)
- added R7: 51k, beepyRcBrd:R_0603_1608Metric_Pad0.98x0.95mm_HandSolder, B.Cu at (82.7, 109.0)
- added R8: 604R, beepyRcBrd:R_0603_1608Metric_Pad0.98x0.95mm_HandSolder, F.Cu at (106.5, 103.0)
- added R9: 150k, beepyRcBrd:R_0603_1608Metric_Pad0.98x0.95mm_HandSolder, F.Cu at (105.5, 88.8)
- added R_FB1: 49k, beepyRcBrd:R_0603_1608Metric_Pad0.98x0.95mm_HandSolder, F.Cu at (87.5, 122.0)
- added R_FB2: 3k, beepyRcBrd:R_0603_1608Metric_Pad0.98x0.95mm_HandSolder, F.Cu at (87.5, 118.0)
- added R_FB3: 3k, beepyRcBrd:R_0603_1608Metric_Pad0.98x0.95mm_HandSolder, F.Cu at (87.5, 116.1)
- added Rs1: 17m, beepyRcBrd:R_1206_3216Metric_Pad1.30x1.75mm_HandSolder, F.Cu at (75.0, 115.5)
- added SW1: SW_Push, beepyRcBrd:SW-SMD_L3.9-W3.0-P4.45, F.Cu at (108.1, 154.0)
- added SW2: SW_Push, beepyRcBrd:SW-SMD_L3.9-W3.0-P4.45, F.Cu at (123.3, 154.0)
- added SW4: SW_Push, beepyRcBrd:SW-SMD_L3.9-W3.0-P4.45, F.Cu at (115.8, 154.0)
- added TP10: TestPoint, beepyRcBrd:TestPoint_Pad_D1.0mm, F.Cu at (87.0, 42.0)
- added TP11: TestPoint, beepyRcBrd:TestPoint_Pad_D1.0mm, F.Cu at (94.2, 108.5)
- added TP12: TestPoint, beepyRcBrd:TestPoint_Pad_D1.0mm, F.Cu at (87.2, 108.5)
- added TP13: TestPoint, beepyRcBrd:TestPoint_Pad_D1.0mm, F.Cu at (121.0, 123.2)
- added TP14: TestPoint, beepyRcBrd:TestPoint_Pad_D1.0mm, F.Cu at (120.0, 116.5)
- added TP2: TestPoint, beepyRcBrd:TestPoint_Pad_D2.5mm, F.Cu at (68.0, 90.5)
- added TP3: TestPoint, beepyRcBrd:TestPoint_Pad_D1.0mm, F.Cu at (116.5, 81.9)
- added TP4: TestPoint, beepyRcBrd:TestPoint_Pad_D1.0mm, F.Cu at (118.6, 81.9)
- added TP7: TestPoint, beepyRcBrd:TestPoint_Pad_D1.0mm, F.Cu at (116.3, 107.5)
- added TP9: TestPoint, beepyRcBrd:TestPoint_Pad_D1.0mm, F.Cu at (82.7, 69.5)
- added U1: TC118S, beepyRcBrd:SOP-8_L4.9-W3.9-P1.27-LS6.0-BL, B.Cu at (79.3, 57.1)
- added U10: CD4011BM96, beepyRcBrd:SOIC-14_L8.7-W3.9-P1.27-LS6.0-BL, B.Cu at (90.5, 105.0)
- added U11: AT25SF161B-SSHB-T, beepyRcBrd:SOP-8_L4.9-W3.9-P1.27-LS6.0-BL, B.Cu at (95.1, 81.2)
- added U12: AT7456ELAH_C42388749, beepyRcBrd:LGA-16_L6.8-W4.0-P0.65-TL-2EP, F.Cu at (86.3, 79.8)
- added U2: STM32F446RETx, beepyRcBrd:LQFP-64_10x10mm_P0.5mm, F.Cu at (117.4, 93.5)
- added U3: INA139, beepyRcBrd:SOT-23-5, B.Cu at (78.2, 117.4)
- added U4: TPS564242DRLR, beepyRcBrd:SOT-5X3-6_W1.6-L1.2-P0.50-LS1.6-BL, F.Cu at (81.7, 112.5)
- added U5: MC33275ST-3.3T3G, beepyRcBrd:SOT-223_L6.5-W3.5-P2.30-LS7.0-BR, B.Cu at (72.9, 135.1)
- added U6: TC118S, beepyRcBrd:SOP-8_L4.9-W3.9-P1.27-LS6.0-BL, B.Cu at (111.9, 56.6)
- added U7: TC118S, beepyRcBrd:SOP-8_L4.9-W3.9-P1.27-LS6.0-BL, B.Cu at (108.4, 140.1)
- added U8: TC118S, beepyRcBrd:SOP-8_L4.9-W3.9-P1.27-LS6.0-BL, B.Cu at (119.7, 140.0)
- added U9: TLV1117-33, beepyRcBrd:SOT-223_L6.5-W3.5-P2.30-LS7.0-BR, B.Cu at (82.7, 135.3)
- added X2: H6OEL89CSC-SUGYLC-27M, beepyRcBrd:HC-49S_L11.4-W4.8-LS12.7, F.Cu at (95.3, 82.8)
- added Y3: HY8M49SSMDOB2R20, beepyRcBrd:CRYSTAL-SMD_L11.4-W4.7-LS12.7, F.Cu at (99.5, 100.3)
- added Y4: M332768DWNAC, beepyRcBrd:OSC-SMD_2P-L7.4-W3.1-LS8.0, F.Cu at (99.5, 86.9)
Routing:
- net V_MOT: track 0.00 -> 280.8 mm, vias 0 -> 25
- net +5V: track 0.00 -> 175.8 mm, vias 0 -> 2
- net /MCU/NRST: track 0.00 -> 153.6 mm, vias 0 -> 4
- net V_3V3_EXT: track 0.00 -> 145.9 mm, vias 0 -> 12
- net V_SERVO: track 0.00 -> 127.9 mm, vias 0 -> 24
- net /RC_RX: track 0.00 -> 117.0 mm, vias 0 -> 3
- net /I2C_SDA: track 0.00 -> 109.0 mm, vias 0 -> 3
- net /LED_G: track 0.00 -> 108.5 mm, vias 0 -> 2
- net /LED_Y: track 0.00 -> 106.7 mm, vias 0 -> 2
- net /B2: track 0.00 -> 104.4 mm, vias 0 -> 2
- net /RC_TX: track 0.00 -> 100.4 mm, vias 0 -> 3
- net GND: track 0.00 -> 99.7 mm, vias 0 -> 95
- net /LED_R: track 0.00 -> 98.7 mm, vias 0 -> 2
- net /BAR_CS: track 0.00 -> 96.2 mm, vias 0 -> 2
- net /SPI_SCK: track 0.00 -> 95.7 mm, vias 0 -> 1
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- added copper zone on F.Cu, net /Power/BatteryMonitor/V_BAT
- added copper zone on B.Cu, net GND
- added copper zone on F.Cu, net GND
- added copper zone on In1.Cu, net GND
- added copper zone on B.Cu, net Net-(D4-Pad2)
- added copper zone on F.Cu, net Net-(D4-Pad2)
- added copper zone on B.Cu, net Net-(D5-K)
- added copper zone on F.Cu, net Net-(U4-SW)
- added copper zone on B.Cu, net V_3V3_EXT
- added copper zone on In2.Cu, net V_3V3_EXT
- added copper zone on F.Cu, net V_BAT
- added copper zone on B.Cu, net V_MCU
- added copper zone on In2.Cu, net V_MCU
- added copper zone on B.Cu, net V_MOT
- added copper zone on F.Cu, net V_MOT
- added copper zone on In2.Cu, net V_MOT
- added copper zone on F.Cu, net V_SERVO
- added copper zone on In2.Cu, net V_SERVO
Other:
- board outline added: 91 x 130 mm
- board text added: "2026/04/15"
- board text added: "3.3V"
- board text added: "3V3"
- board text added: "3V3_EXT"
- board text added: "5V"
- board text added: "5V IN"
- board text added: "ANCS"
- board text added: "B1"
- board text added: "B2"
- board text added: "BCS"
- board text added: "BOOT0"
- board text added: "BeepyRC"
- board text added: "BeepyRcBrd Rev. 0.0"
- board text added: "Debug"
- board text added: "Dimensions in mm"
- board text added: "E3.3V"
- board text added: "EN 3V3_EXT"
- board text added: "ENCA"
- board text added: "ENCB"
- board text added: "ElectronPlant"
- board text added: "ElectronPlant/beepy_rc"
- board text added: "GND"
- board text added: "GNSS Power"
- board text added: "I2C"
- board text added: "I2C Power"
- board text added: "L1"
- board text added: "L2"
- board text added: "L3"
- board text added: "Lights"
- board text added: "MISO"
- board text added: "MOSI"
- board text added: "NC"
- board text added: "NRST"
- board text added: "PPS"
- board text added: "PWM"
- board text added: "PWMA"
- board text added: "PWMB"
- board text added: "Power Output"
- board text added: "RST"
- board text added: "Rx IN"
- board text added: "S1"
- board text added: "S2"
- board text added: "S3"
- board text added: "SCK"
- board text added: "SCL"
- board text added: "SDA"
- board text added: "SERVOS"
- board text added: "SPI/IMU"
- board text added: "SWCL"
- board text added: "SWDIO"
- board text added: "SWO"
- board text added: "Serial/GNSS"
- board text added: "Tx IN"
- board text added: "V+"
- board text added: "VBAT"
- board text added: "VID_I"
- board text added: "VID_O"
- board text added: "VMCU"
- board text added: "VTX"
- board text added: "V_MCU"
- board text added: "© David Arnaiz 2026 Licensed under CERN-OHL-S v2"
