File: hardware/beepyRcBrd/buck_converter.kicad_sch (KiCad schematic)
At the start: 19 parts, among them Q3 BSS138DW-7-F, U10 CD4011BM96, U4 TPS564242DRLR

Commit message: feat: completed beepyRcBrd_rev_0_0.pdf
Parts:
- C10, C12, C13, C6, C7, C8, C9: footprint Capacitor_SMD:C_0603_1608Metric_Pad1.08x0.95mm_HandSolder -> beepyRcBrd:C_0603_1608Metric_Pad1.08x0.95mm_HandSolder
- L2: footprint lscs:IND-SMD_L7.0-W6.6_MCW-0650-220 -> beepyRcBrd:IND-SMD_L7.0-W6.6_MCW-0650-220
- Q3: footprint lscs:SC-70-6_L2.2-W1.3-P0.65-LS2.1-TL -> beepyRcBrd:SC-70-6_L2.2-W1.3-P0.65-LS2.1-TL
- R10, R12, R7, R_FB1, R_FB2, R_FB3: footprint Resistor_SMD:R_0603_1608Metric_Pad0.98x0.95mm_HandSolder -> beepyRcBrd:R_0603_1608Metric_Pad0.98x0.95mm_HandSolder
- R44: renamed from R_EN1; value 50k -> 51k; footprint Resistor_SMD:R_0603_1608Metric_Pad0.98x0.95mm_HandSolder -> beepyRcBrd:R_0603_1608Metric_Pad0.98x0.95mm_HandSolder
- R45: renamed from R_EN2; footprint Resistor_SMD:R_0603_1608Metric_Pad0.98x0.95mm_HandSolder -> beepyRcBrd:R_0603_1608Metric_Pad0.98x0.95mm_HandSolder
- U10: footprint lscs:SOIC-14_L8.7-W3.9-P1.27-LS6.0-BL -> beepyRcBrd:SOIC-14_L8.7-W3.9-P1.27-LS6.0-BL
- U4: footprint lscs:SOT-5X3-6_W1.6-L1.2-P0.50-LS1.6-BL -> beepyRcBrd:SOT-5X3-6_W1.6-L1.2-P0.50-LS1.6-BL
Changed lines of the file:
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@@
 		(rev "V0.0")
 		(company "Electron Plant")
+		(comment 1 "© David Arnaiz 2026")
+		(comment 2 "Licensed under CERN-OHL-S v2")
 	)
 	(text "0.1%"
@@
 	(text "BeepyRC"
 		(exclude_from_sim no)
-		(at 232.664 173.99 0)
+		(at 251.206 174.498 0)
 		(effects
 			(font
@@
 			)
 		)
-		(property "Footprint" "Capacitor_SMD:C_0603_1608Metric_Pad1.08x0.95mm_HandSolder"
+		(property "Footprint" "beepyRcBrd:C_0603_1608Metric_Pad1.08x0.95mm_HandSolder"
 			(at 119.0752 104.14 0)
 			(effects
@@
 			)
 		)
-		(property "Footprint" "Capacitor_SMD:C_0603_1608Metric_Pad1.08x0.95mm_HandSolder"
+		(property "Footprint" "beepyRcBrd:C_0603_1608Metric_Pad1.08x0.95mm_HandSolder"
 			(at 221.9452 40.64 0)
 			(effects
@@
 			)
 		)
-		(property "Footprint" "Capacitor_SMD:C_0603_1608Metric_Pad1.08x0.95mm_HandSolder"
+		(property "Footprint" "beepyRcBrd:C_0603_1608Metric_Pad1.08x0.95mm_HandSolder"
 			(at 152.0952 48.26 0)
 			(effects
@@
 			)
 		)
-		(property "Footprint" "Capacitor_SMD:C_0603_1608Metric_Pad1.08x0.95mm_HandSolder"
+		(property "Footprint" "beepyRcBrd:C_0603_1608Metric_Pad1.08x0.95mm_HandSolder"
 			(at 162.2552 48.26 0)
 			(effects
@@
 			)
 		)
-		(property "Footprint" "Resistor_SMD:R_0603_1608Metric_Pad0.98x0.95mm_HandSolder"
+		(property "Footprint" "beepyRcBrd:R_0603_1608Metric_Pad0.98x0.95mm_HandSolder"
 			(at 242.062 27.94 90)
 			(effects
@@
 			)
 		)
-		(property "Footprint" "Resistor_SMD:R_0603_1608Metric_Pad0.98x0.95mm_HandSolder"
+		(property "Footprint" "beepyRcBrd:R_0603_1608Metric_Pad0.98x0.95mm_HandSolder"
 			(at 46.482 71.12 90)
 			(effects
@@
 			)
 		)
-		(property "Footprint" "Resistor_SMD:R_0603_1608Metric_Pad0.98x0.95mm_HandSolder"
+		(property "Footprint" "beepyRcBrd:R_0603_1608Metric_Pad0.98x0.95mm_HandSolder"
 			(at 129.54 97.028 90)
 			(effects
@@
 			)
 		)
-		(property "Footprint" "Capacitor_SMD:C_0603_1608Metric_Pad1.08x0.95mm_HandSolder"
+		(property "Footprint" "beepyRcBrd:C_0603_1608Metric_Pad1.08x0.95mm_HandSolder"
 			(at 172.4152 48.26 0)
 			(effects
@@
 		(dnp no)
 		(fields_autoplaced yes)
-		(property "Reference" "R_EN1"
+		(property "Reference" "R44"
 			(at 125.73 40.6399 0)
 			(effects
@@
 			)
 		)
-		(property "Value" "50k"
+		(property "Value" "51k"
 			(at 125.73 43.1799 0)
 			(effects
@@
 			)
 		)
-		(property "Footprint" "Resistor_SMD:R_0603_1608Metric_Pad0.98x0.95mm_HandSolder"
+		(property "Footprint" "beepyRcBrd:R_0603_1608Metric_Pad0.98x0.95mm_HandSolder"
 			(at 121.412 41.91 90)
 			(effects
@@
 			(project "beepyRcBrd"
 				(path "/c17d25e0-24c9-466a-aee2-e4b5dcf71363/25416242-1327-4080-bdb9-7e497d324eea/8dd0d8ba-da84-4cf7-b2c1-68376c83e89b"
-					(reference "R_EN1")
+					(reference "R44")
 					(unit 1)
 				)
@@
 			)
 		)
-		(property "Footprint" "Capacitor_SMD:C_0603_1608Metric_Pad1.08x0.95mm_HandSolder"
+		(property "Footprint" "beepyRcBrd:C_0603_1608Metric_Pad1.08x0.95mm_HandSolder"
 			(at 233.3752 40.64 0)
 			(effects
@@
 			)
 		)
-		(property "Footprint" "lscs:SC-70-6_L2.2-W1.3-P0.65-LS2.1-TL"
+		(property "Footprint" "beepyRcBrd:SC-70-6_L2.2-W1.3-P0.65-LS2.1-TL"
 			(at 91.44 105.41 0)
 			(effects
@@
 			)
 		)
-		(property "Footprint" "Resistor_SMD:R_0603_1608Metric_Pad0.98x0.95mm_HandSolder"
+		(property "Footprint" "beepyRcBrd:R_0603_1608Metric_Pad0.98x0.95mm_HandSolder"
 			(at 242.062 54.61 90)
 			(effects
@@
 			)
 		)
-		(property "Footprint" "Resistor_SMD:R_0603_1608Metric_Pad0.98x0.95mm_HandSolder"
+		(property "Footprint" "beepyRcBrd:R_0603_1608Metric_Pad0.98x0.95mm_HandSolder"
 			(at 242.062 44.45 90)
 			(effects
@@
 			)
 		)
-		(property "Footprint" "lscs:SOT-5X3-6_W1.6-L1.2-P0.50-LS1.6-BL"
+		(property "Footprint" "beepyRcBrd:SOT-5X3-6_W1.6-L1.2-P0.50-LS1.6-BL"
 			(at 194.31 48.26 0)
 			(effects
@@
 			)
 		)
-		(property "Footprint" "lscs:SOIC-14_L8.7-W3.9-P1.27-LS6.0-BL"
+		(property "Footprint" "beepyRcBrd:SOIC-14_L8.7-W3.9-P1.27-LS6.0-BL"
 			(at 91.44 76.2 0)
 			(effects
@@
 			)
 		)
-		(property "Footprint" "Capacitor_SMD:C_0603_1608Metric_Pad1.08x0.95mm_HandSolder"
+		(property "Footprint" "beepyRcBrd:C_0603_1608Metric_Pad1.08x0.95mm_HandSolder"
 			(at 65.7352 62.23 0)
 			(effects
@@
 		(dnp no)
 		(fields_autoplaced yes)
-		(property "Reference" "R_EN2"
+		(property "Reference" "R45"
 			(at 125.73 62.2299 0)
 			(effects
@@
 			)
 		)
-		(property "Footprint" "Resistor_SMD:R_0603_1608Metric_Pad0.98x0.95mm_HandSolder"
+		(property "Footprint" "beepyRcBrd:R_0603_1608Metric_Pad0.98x0.95mm_HandSolder"
 			(at 121.412 63.5 90)
 			(effects
@@
 			(project "beepyRcBrd"
 				(path "/c17d25e0-24c9-466a-aee2-e4b5dcf71363/25416242-1327-4080-bdb9-7e497d324eea/8dd0d8ba-da84-4cf7-b2c1-68376c83e89b"
-					(reference "R_EN2")
+					(reference "R45")
 					(unit 1)
 				)
@@
 			)
 		)
-		(property "Footprint" "lscs:IND-SMD_L7.0-W6.6_MCW-0650-220"
+		(property "Footprint" "beepyRcBrd:IND-SMD_L7.0-W6.6_MCW-0650-220"
 			(at 194.31 21.59 0)
 			(effects
@@
 			)
 		)
-		(property "Footprint" "Resistor_SMD:R_0603_1608Metric_Pad0.98x0.95mm_HandSolder"
+		(property "Footprint" "beepyRcBrd:R_0603_1608Metric_Pad0.98x0.95mm_HandSolder"
 			(at 62.992 44.45 90)
 			(effects
