File: hardware/beepyRcBrd/io.kicad_sch (KiCad schematic)
At the start: 32 parts, among them J12 Conn_01x05, J14 Conn_01x04, J18 Conn_01x04, J8 Conn_01x08, Q1 BSS138LT1G, Q2 BSS138LT1G, Q5 BSS138LT1G, SW1 SW_Push, SW4 SW_Push

Commit message: fix: net names
Parts:
- added TP2: TestPoint, TestPoint:TestPoint_Pad_D2.5mm, symbol beepyRc_symbols:TestPoint
Connections:
- new net ACC_INT: TP2.1
Other:
- note added: "Potential Rework to connect the interrupt pin"
- moved on the sheet: J8, R1, R26

Commit message: fix: passing schematics ERC rules
Parts:
- J14: footprint TestPoint:TestPoint_Bridge_Pitch2.54mm_Drill1.0mm -> (none)
Connections:
- net 3V3_EXT renamed V_3V3_EXT
- net V_LIGHTS renamed V_SERVO
Other:
- moved on the sheet: R28

Commit message: feat: completed beepyRcBrd_rev_0_0.pdf
Parts:
- removed J12: Conn_01x05, TestPoint:TestPoint_Bridge_Pitch2.54mm_Drill1.0mm, symbol beepyRc_symbols:Conn_01x05
- added H13, H14: MT, beepyRcBrd:MountingHole_4.3mm_M4_DIN965_Pad_TopBottom, symbol beepyRc_symbols:MountingHole_Pad
- added J4: Conn_01x06, beepyRcBrd:PinHeader_1x06_P2.54mm_Vertical, symbol beepyRc_symbols:Conn_01x06
- BUZZER1: footprint lscs:BUZ-TH_BD12.0-P7.60-D0.6-FD -> beepyRcBrd:BUZ-TH_BD12.0-P7.60-D0.6-FD
- D1, D2, D3: footprint LED_SMD:LED_0603_1608Metric_Pad1.05x0.95mm_HandSolder -> beepyRcBrd:LED_0603_1608Metric_Pad1.05x0.95mm_HandSolder
- D6, D8: footprint lscs:SOT-23_L2.9-W1.3-P1.90-LS2.4-BR -> beepyRcBrd:SOT-23_L2.9-W1.3-P1.90-LS2.4-BR
- D9: footprint lscs:SOT-723_L1.2-W0.8-P0.40-LS1.2-BR -> beepyRcBrd:SOT-723_L1.2-W0.8-P0.40-LS1.2-BR; now not fitted
- J14: footprint (none) -> beepyRcBrd:PinHeader_1x04_P2.54mm_Vertical
- J18: footprint TestPoint:TestPoint_Bridge_Pitch2.54mm_Drill1.0mm -> beepyRcBrd:PinHeader_1x04_P2.54mm_Vertical
- J8: footprint TestPoint:TestPoint_Bridge_Pitch2.54mm_Drill1.0mm -> beepyRcBrd:gy91
- Q1, Q2, Q5: footprint lscs:SOT-23-3_L2.9-W1.6-P1.90-LS2.8-BR -> beepyRcBrd:SOT-23-3_L2.9-W1.6-P1.90-LS2.8-BR
- R1, R13, R15, R17, R18, R2, R26, R27, R28, R29, R3, R30, R31, R4, R5, R6: footprint Resistor_SMD:R_0603_1608Metric_Pad0.98x0.95mm_HandSolder -> beepyRcBrd:R_0603_1608Metric_Pad0.98x0.95mm_HandSolder
- SW1, SW4: footprint lscs:SW-SMD_L3.9-W3.0-P4.45 -> beepyRcBrd:SW-SMD_L3.9-W3.0-P4.45
- TP2: footprint TestPoint:TestPoint_Pad_D2.5mm -> beepyRcBrd:TestPoint_Pad_D2.5mm
Connections:
- net GND: now also H13.1, H14.1, J4.3 (Pin_3)
- net GNSS_PPS: now also J4.6 (Pin_6)
- net GNSS_RX: now also J4.5 (Pin_5)
- net GNSS_TX: now also J4.4 (Pin_4)
- net at R13.2, R15.2: now also J4.2 (Pin_2)
- new net V_USB: J4.1 (Pin_1)
Other:
- note added: "Mounting Holes"
- moved on the sheet: R13, R15
