File: hardware/beepyRcBrd/mcu.kicad_sch (KiCad schematic)
At the start: 33 parts, among them J13 Conn_01x04, J3 Conn_01x06, J4 Conn_01x02_Pin, SW2 SW_Push, U11 AT25SF161B-SSHB-T, U2 STM32F446RETx, Y3 HY8M49SSMDOB2R20, Y4 M332768DWNAC

Commit message: fix: passing schematics ERC rules
Connections:
- net SPI_MISO is gone; now on net SPI2_MISO: R23.1
Other:
- note added: "ESR <1Ω"
Changed lines of the file:
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@@
 		)
 	)
+	(text "ESR <1Ω"
+		(exclude_from_sim no)
+		(at 95.758 124.714 0)
+		(effects
+			(font
+				(size 1.27 1.27)
+			)
+		)
+	)
 	(text "- 10uF ceramic cap for the package.\n- 100nF ceramic between pins 18-19, 31-32, 47-48 and 63-64.\n- Vbat on pin 1 is connected to VDD with a 100nF decoupling cap.\n- VDDA is connected to VDD through a ferrite bead.\n- VDDA is decoupled with a 1uF and a 100nF cap between pins 12-13.\n- GNDA is directly connected to the GND ground plane."
 		(exclude_from_sim no)
@@
 		)
 	)
-	(label "SPI_MISO"
+	(label "SPI2_MISO"
 		(at 55.88 175.26 0)
 		(effects
@@
 		)
 	)
-	(label "ESR <1Ω"
-		(at 91.44 125.73 0)
-		(effects
-			(font
-				(size 1.27 1.27)
-			)
-			(justify left bottom)
-		)
-	)
 	(label "SWDIO"
 		(at 251.46 149.86 0)
@@
 	)
 	(symbol
+		(lib_id "beepyRc_symbols:VDDA")
+		(at 270.51 20.32 0)
+		(unit 1)
+		(exclude_from_sim no)
+		(in_bom yes)
+		(on_board yes)
+		(dnp no)
+		(property "Reference" "#PWR0136"
+			(at 270.51 24.13 0)
+			(effects
+				(font
+					(size 1.27 1.27)
+				)
+				(hide yes)
+			)
+		)
+		(property "Value" "VDDA"
+			(at 270.51 16.51 0)
+			(effects
+				(font
+					(size 1.27 1.27)
+				)
+			)
+		)
+		(property "Footprint" ""
+			(at 270.51 20.32 0)
+			(effects
+				(font
+					(size 1.27 1.27)
+				)
+				(hide yes)
+			)
+		)
+		(property "Datasheet" ""
+			(at 270.51 20.32 0)
+			(effects
+				(font
+					(size 1.27 1.27)
+				)
+				(hide yes)
+			)
+		)
+		(property "Description" "Power symbol creates a global label with name \"VDDA\""
+			(at 270.51 20.32 0)
+			(effects
+				(font
+					(size 1.27 1.27)
+				)
+				(hide yes)
+			)
+		)
+		(pin "1"
+		)
+		(instances
+			(project "beepyRcBrd"
+				(path "/c17d25e0-24c9-466a-aee2-e4b5dcf71363/12039923-f6f3-42f8-83b6-663c3bf7be39"
+					(reference "#PWR0136")
+					(unit 1)
+				)
+			)
+		)
+	)
+	(symbol
 		(lib_id "beepyRc_symbols:C")
 		(at 224.79 39.37 0)
@@
 					(unit 1)
 				)
+			)
+		)
+	)
+	(symbol
+		(lib_id "beepyRc_symbols:PWR_FLAG")
+		(at 270.51 20.32 180)
+		(unit 1)
+		(exclude_from_sim no)
+		(in_bom yes)
+		(on_board yes)
+		(dnp no)
+		(fields_autoplaced yes)
+		(property "Reference" "#FLG04"
+			(at 270.51 22.225 0)
+			(effects
+				(font
+					(size 1.27 1.27)
+				)
+				(hide yes)
+			)
+		)
+		(property "Value" "PWR_FLAG"
+			(at 273.05 21.5899 0)
+			(effects
+				(font
+					(size 1.27 1.27)
+				)
+				(justify right)
+			)
+		)
+		(property "Footprint" ""
+			(at 270.51 20.32 0)
+			(effects
+				(font
+					(size 1.27 1.27)
+				)
+				(hide yes)
+			)
+		)
+		(property "Datasheet" "~"
+			(at 270.51 20.32 0)
+			(effects
+				(font
+					(size 1.27 1.27)
+				)
+				(hide yes)
+			)
+		)
+		(property "Description" "Special symbol for telling ERC where power comes from"
+			(at 270.51 20.32 0)
+			(effects
+				(font
+					(size 1.27 1.27)
+				)
+				(hide yes)
+			)
+		)
+		(pin "1"
+		)
+		(instances
+			(project "beepyRcBrd"
+				(path "/c17d25e0-24c9-466a-aee2-e4b5dcf71363/12039923-f6f3-42f8-83b6-663c3bf7be39"
+					(reference "#FLG04")
+					(unit 1)
+				)

Commit message: feat: completed beepyRcBrd_rev_0_0.pdf
Parts:
- removed J13: Conn_01x04, TestPoint:TestPoint_Bridge_Pitch2.54mm_Drill1.0mm, symbol beepyRc_symbols:Conn_01x04
- removed J4: Conn_01x02_Pin, TestPoint:TestPoint_Bridge_Pitch2.54mm_Drill1.0mm, symbol beepyRc_symbols:Conn_01x02_Pin
- removed R21, R22: 0, Resistor_SMD:R_0603_1608Metric_Pad0.98x0.95mm_HandSolder, symbol beepyRc_symbols:R
- added TP3, TP4: TestPoint, beepyRcBrd:TestPoint_Pad_D1.0mm, symbol beepyRc_symbols:TestPoint
- C15, C16, C17, C18, C19, C20, C21, C22, C23, C24, C25, C26, C27, C28: footprint Capacitor_SMD:C_0603_1608Metric_Pad1.08x0.95mm_HandSolder -> beepyRcBrd:C_0603_1608Metric_Pad1.08x0.95mm_HandSolder
- FB2, R14, R19, R23, R24, R25, R32, R8, R9: footprint Resistor_SMD:R_0603_1608Metric_Pad0.98x0.95mm_HandSolder -> beepyRcBrd:R_0603_1608Metric_Pad0.98x0.95mm_HandSolder
- J3: footprint TestPoint:TestPoint_Bridge_Pitch2.54mm_Drill1.0mm -> beepyRcBrd:PinHeader_1x06_P2.54mm_Vertical
- SW2: footprint lscs:SW-SMD_L3.9-W3.0-P4.45 -> beepyRcBrd:SW-SMD_L3.9-W3.0-P4.45
- U11: footprint lscs:SOP-8_L4.9-W3.9-P1.27-LS6.0-BL -> beepyRcBrd:SOP-8_L4.9-W3.9-P1.27-LS6.0-BL
- U2: footprint Package_QFP:LQFP-64_10x10mm_P0.5mm -> beepyRcBrd:LQFP-64_10x10mm_P0.5mm
- Y3: footprint lscs:CRYSTAL-SMD_L11.4-W4.7-LS12.7 -> beepyRcBrd:CRYSTAL-SMD_L11.4-W4.7-LS12.7
- Y4: footprint lscs:OSC-SMD_2P-L7.4-W3.1-LS8.0 -> beepyRcBrd:OSC-SMD_2P-L7.4-W3.1-LS8.0
Connections:
- net DBG_RX is gone; now on net UART2_RX: U2.17 (PA3)
- net DBG_TX is gone; now on net UART2_TX: U2.16 (PA2)
- net BOOT0: now also TP4.1
- net V_MCU: now also TP3.1
Other:
- note removed: "Debug Serial is shared"
- moved on the sheet: J3
