File: hardware/beepyRcBrd/power.kicad_sch (KiCad schematic)
At the start: 25 parts

Commit message: fix: passing schematics ERC rules
Connections:
- net V_LIGHTS renamed V_SERVO
Changed lines of the file:
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@@
-	(wire
-		(pts
-			(xy 173.99 54.61) (xy 173.99 50.8)
-		)
-		(stroke
-			(width 0)
-			(type default)
-		)
-	)
 	(wire
 		(pts
@@
 	(wire
 		(pts
-			(xy 177.8 54.61) (xy 173.99 54.61)
-		)
-		(stroke
-			(width 0)
-			(type default)
-		)
-	)
-	(wire
-		(pts
 			(xy 30.48 173.99) (xy 34.29 173.99)
 		)
@@
 		)
 	)
-	(hierarchical_label "V_LIGHTS"
-		(shape output)
-		(at 177.8 54.61 0)
-		(effects
-			(font
-				(size 1.27 1.27)
-			)
-			(justify left)
-		)
-	)

Commit message: feat: completed beepyRcBrd_rev_0_0.pdf
Parts:
- removed H1, H2, H3, H4: MT, MountingHole:MountingHole_4.3mm_M4_DIN965_Pad_TopBottom, symbol beepyRc_symbols:MountingHole_Pad
- removed H10, H11, H12, H5, H6, H7, H8, H9: MT, MountingHole:MountingHole_3mm_Pad_TopBottom, symbol beepyRc_symbols:MountingHole_Pad
- removed TP8: TestPoint, TestPoint:TestPoint_Pad_D1.0mm, symbol beepyRc_symbols:TestPoint
- D4: footprint lscs:SOT-23-3_L2.9-W1.6-P1.90-LS2.8-BR -> beepyRcBrd:SOT-23-3_L2.9-W1.6-P1.90-LS2.8-BR
- D7: footprint lscs:SMB_L4.6-W3.6-LS5.3-RD -> beepyRcBrd:SMB_L4.6-W3.6-LS5.3-RD
- F1, F2: footprint Fuse:Fuse_1812_4532Metric_Pad1.30x3.40mm_HandSolder -> beepyRcBrd:Fuse_1812_4532Metric_Pad1.30x3.40mm_HandSolder
- FB1: footprint Resistor_SMD:R_0603_1608Metric_Pad0.98x0.95mm_HandSolder -> beepyRcBrd:R_0603_1608Metric_Pad0.98x0.95mm_HandSolder
- TP10, TP11, TP12, TP13, TP14, TP7, TP9: footprint TestPoint:TestPoint_Pad_D1.0mm -> beepyRcBrd:TestPoint_Pad_D1.0mm
Other:
- note removed: "Board Mounting Holes"
- note removed: "Motor Mounting Holes"
